File: thinkpad.kicad_pcb (KiCad board)
At the start: 2 copper layers, 287 x 109 mm, 127 parts, among them J1 Conn_01x06_MountingPin, J2 Conn_01x20_Socket, J3 Conn_01x06_Socket, J4 Conn_01x04_Pin, SW1 SW_Push, U1 Raspberry_Pi_Pico

Commit message: Give 3V3 to touchpad
Parts:
- added G***: LOGO, libmodulo:ModuloIndustries_logo, F.Cu at (317.1, 152.7)
- J4: value Conn_01x04_Pin -> Touchpad_Conn
Connections:
- J4 pad 4: VCC -> 3V3
- U1 pad 36: unconnected-(U1-3V3-Pad36) -> 3V3
Routing:
- net 3V3: track 0.00 -> 77.3 mm, vias 0 -> 1
- net VCC: track 99.7 -> 77.4 mm
Other:
- board text added: "X"

Commit message: Fix issue with usb and aligning the tape
Parts:
- removed JP1: SolderJumper_3_Open, Jumper:SolderJumper-3_P1.3mm_Open_Pad1.0x1.5mm_NumberLabels
- removed SW1: SW_Push, Button_Switch_THT:SW_PUSH-12mm
- added S61: Keyswitch, ScottoKeebs_Choc:Choc_Mini_1.00u, F.Cu at (190.6, 58.7)
- J1: moved to B.Cu
- moved J1 8.40 mm to (211.0, 151.9), turned to 180 degrees
- moved J4 2.73 mm to (229.6, 156.0)
- moved J2 0.80 mm to (221.1, 54.1)
Connections:
- J3 pad 2: USB- -> USB+
- J3 pad 3: USB+ -> USB-
- U1 pad 3: Net-(SW1-Pad1) -> GND
Routing:
- net Net-(SW1-Pad1): track 61.9 -> 0.00 mm
- net SC_DTCT: track 20.4 -> 0.00 mm, vias 2 -> 0
- net USB-: track 80.2 -> 61.2 mm, vias 2 -> 1
- net USB+: track 78.2 -> 62.1 mm, vias 1 -> 0
- net VCC: track 77.4 -> 67.6 mm, vias 1 -> 2
- net Net-(J2-Pin_7): track 130.5 -> 122.7 mm
- net 3V3: track 77.3 -> 74.5 mm, vias 1 -> 3
- net GND: track 5.57 -> 4.02 mm
- net SDA: track 42.4 -> 41.7 mm
- net SCL: track 46.8 -> 46.3 mm
Other:
- outline, holes or cut-outs redrawn

Commit message: Change switches
Parts:
- added F1: Fuse, Fuse:Fuse_0805_2012Metric, B.Cu at (195.5, 138.6)
- added J5: Alt_USB, Connector_PinHeader_2.54mm:PinHeader_1x04_P2.54mm_Vertical, F.Cu at (225.2, 70.6)
- added JP1: PowerPin_Jumper_Reverse, Jumper:SolderJumper-2_P1.3mm_Open_Pad1.0x1.5mm, F.Cu at (195.4, 57.8)
- added JP2: PowerPin_Jumper, Jumper:SolderJumper-2_P1.3mm_Open_Pad1.0x1.5mm, F.Cu at (196.9, 53.3)
- D1: footprint ScottoKeebs_Components:Diode_DO-35 -> thinkpad-keyboard:Diode_SMD_THT2; moved to B.Cu
- D10, D11, D12, D13, D14, D15, D16, D17, D18, D19, D2, D20, D21, D22, D23, D24, D25, D26, D27, D28, D29, D3, D30, D31, D32, D33, D34, D35, D36, D37, D38, D39, D4, D40, D41, D42, D43, D44, D45, D46, D47, D48, D49, D5, D50, D51, D52, D53, D54, D55, D56, D57, D58, D59, D6, D60, D7, D8, D9: footprint ScottoKeebs_Components:Diode_DO-35 -> thinkpad-keyboard:Diode_SMD_THT2
- S1, S10, S11, S12, S13, S14, S15, S16, S17, S18, S19, S2, S20, S21, S22, S23, S24, S25, S26, S27, S28, S29, S3, S30, S31, S32, S33, S34, S35, S36, S37, S38, S39, S4, S40, S41, S42, S43, S44, S45, S46, S47, S48, S49, S5, S50, S51, S52, S53, S54, S55, S56, S57, S58, S59, S6, S60, S61, S7, S8, S9: footprint ScottoKeebs_Choc:Choc_Mini_1.00u -> kailh-pg1425-x-switch:Kailh-PG1425-X-Switch
- moved S61 55.2 mm to (244.2, 45.3), turned to 10 degrees
- moved D7 14.9 mm to (79.6, 60.5)
- moved D19 14.9 mm to (73.7, 94.0)
- moved D3 14.9 mm to (118.0, 50.0)
- moved D28 14.9 mm to (123.9, 120.1)
- moved D27 14.9 mm to (106.2, 117.0)
- moved D13 14.9 mm to (76.6, 77.3)
- moved D15 14.9 mm to (112.1, 83.5)
- moved D4 14.9 mm to (135.7, 53.2)
- moved D9 14.9 mm to (115.0, 66.8)
- moved D12 14.9 mm to (168.2, 76.2)
- moved D22 14.9 mm to (126.8, 103.4)
- moved D26 14.9 mm to (88.4, 113.9)
- moved D1 14.9 mm to (82.5, 43.8)
- moved D30 14.9 mm to (159.3, 126.4)
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Connections:
- J1 pad 1: SC_DTCT -> Net-(J1-Pin_1)
- J1 pad 2: unconnected-(J1-Pin_2-Pad2) -> USB-
- J1 pad 3: GND -> USB+
- J1 pad 4: USB+ -> GND
- J1 pad 5: USB- -> unconnected-(J1-Pin_5-Pad5)
- J1 pad 6: VCC -> GND
- J2 pad 14: unconnected-(J2-Pin_14-Pad14) -> Net-(J2-Pin_14)
- S61 pad 1: Net-(J2-Pin_7) -> Net-(JP1-A)
- U1 pad 20: Net-(J2-Pin_7) -> Net-(JP1-A)
Routing:
- net Net-(JP1-A): track 0.00 -> 155.4 mm, vias 0 -> 1
- net Net-(J2-Pin_7): track 122.7 -> 14.9 mm, vias 1 -> 0
- net Row 4: track 289.3 -> 343.6 mm, vias 0 -> 1
- net Row 1: track 271.5 -> 324.3 mm, vias 0 -> 1
- net Row 0: track 292.7 -> 345.5 mm
- net Row 3: track 270.9 -> 323.1 mm, vias 0 -> 1
- net Row 2: track 261.0 -> 312.0 mm, vias 0 -> 1
- net Col 8: track 180.6 -> 145.5 mm
- net Col 9: track 192.9 -> 160.2 mm
- net Col 7: track 173.8 -> 141.4 mm
- net Net-(J2-Pin_14): track 0.00 -> 31.9 mm
- net USB+: track 62.1 -> 86.7 mm, vias 0 -> 2
- net USB-: track 61.2 -> 84.1 mm
- net Col 6: track 153.5 -> 134.7 mm
- net Col 11: track 228.6 -> 215.0 mm
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Other:
- outline, holes or cut-outs redrawn
- board text added: "K"
- board text added: "Keyboard tape"
- board text added: "Mount"
- board text added: "Solder"
- board text added: "Touchpad I2C"
- board text added: "USB Alt"

Commit message: Fix issues and add breakable touchpad
Parts:
- moved J1 18.3 mm to (184.9, 133.7)
- moved J4 13.4 mm to (228.7, 136.9)
- moved F1 11.0 mm to (190.7, 128.7), turned to 0 degrees
- moved D59 2.68 mm to (330.6, 96.0)
- moved S15 2.68 mm to (121.5, 86.4)
- moved S32 2.68 mm to (248.6, 78.0)
- moved S41 2.68 mm to (281.1, 55.0)
- moved D25 2.68 mm to (68.1, 110.2)
- moved D31 2.68 mm to (233.1, 61.4)
- moved D54 2.68 mm to (312.9, 99.2)
- moved S12 2.68 mm to (177.6, 79.0)
- moved S21 2.68 mm to (118.5, 103.1)
- moved S22 2.68 mm to (136.2, 106.3)
- moved S36 2.68 mm to (263.4, 58.2)
- moved D41 2.68 mm to (268.6, 55.2)
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Routing:
- net USB+: track 86.7 -> 100.3 mm, vias 2 -> 0
- net USB-: track 84.1 -> 96.7 mm
- net SCL: track 46.3 -> 53.5 mm
- net 3V3: track 74.5 -> 80.9 mm, vias 3 -> 2
- net VCC: track 80.7 -> 85.4 mm
- net Net-(J1-Pin_1): track 9.89 -> 6.48 mm, vias 2 -> 0
- net Col 2: track 187.8 -> 185.4 mm
- net Col 0: track 225.8 -> 223.5 mm
- net Col 1: track 207.9 -> 205.8 mm
- net SDA: track 41.7 -> 40.3 mm
- net Col 10: track 195.8 -> 197.1 mm
- net GND: track 6.89 -> 5.92 mm
Other:
- board size 287 x 109 mm -> 287 x 119.7 mm
- board text removed: "Touchpad I2C"
