File: thinkpad.kicad_pcb (KiCad board)
At the start: 2 copper layers, 287 x 119.7 mm, 131 parts, among them J1 Conn_01x06_MountingPin, J2 Conn_01x20_Socket, J3 Conn_01x06_Socket, J4 Touchpad_Conn, J5 Alt_USB, U1 Raspberry_Pi_Pico

Commit message: filled zones set to no-island, vias added to make ground fills appear in more places (mostly aesthetic), keeb connector duuplicated, drc clean, unconnected 0, life is good
Parts:
- added J6: Conn_01x20_Socket, thinkpad-keyboard:Thinkpad-keyboard-fpc, B.Cu at (208.3, 44.1)
Connections:
- net Net-(J1-Pin_1) renamed VCC_FUSE
Routing:
- net Net-(J2-Pin_7): track 14.9 -> 17.6 mm, vias 0 -> 1
- net Net-(J2-Pin_14): track 31.9 -> 34.1 mm, vias 0 -> 1
- net GND: vias 0 -> 39

Commit message: Update BOM
Other:
- board size 287 x 119.7 mm -> 300.8 x 119.7 mm
- board text added: "V-CUT"
- board text removed: "K"
